File: Hw/PCB_resistive_sensors.kicad_sch (KiCad schematic)
At the start: 56 parts, among them J1 Conn_01x02, J2 Conn_Right, P1 USB_C_Plug_USB2.0, SW1 SW_Push, U1 RP2040, U2 NCP1117ST33T3G, U3 W25Q128JVS, Y1 Crystal

Commit message: anotate changes
Parts:
- removed JP11, JP12: Jp, symbol Jumper:Jumper_2_Open
- removed R19, R20: 22M, Resistor_SMD:R_0805_2012Metric, symbol Device:R
- R13: value DNF -> DNP
Other:
- note added: "I2C SPI -SS combinado con GPIO Serial 2 - GPIO change to W25Q16JVSNIQ"
